File: Spectrogram flex pcb/Spectrogram flex pcb.kicad_sch (KiCad schematic)
At the start: 10 parts

Commit message: Updating Flex PCB
Changed lines of the file:
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@@
-	(wire
-		(pts
-			(xy 125.73 96.52) (xy 125.73 99.06)
-		)
-		(stroke
-			(width 0)
-			(type default)
-		)
-	)
 	(wire
 		(pts
@@
 			)
 		)
-		(pin "2"
-		)
 		(pin "1"
 		)
@@
 			)
 		)
-		(pin "2"
-		)
 		(pin "1"
